File: Raspberry_Pi_2m_TX_LPF_7Stage.sch (KiCad schematic (older format))
At the start: 28 parts, among them J3 RPi_GPIO, P1 3Sip100, P2 4Sip200, P3 2Sip200, P4 SMA, P5 CONN_01X02, Q1 BC817-40, U1 L4940V5 1.5A

Commit message: Board is now compleate
Added second filter
Parts:
- added C7: 10nf, Capacitors_SMD:C_0805_HandSoldering, symbol C_Small
- added F1: LFCN-80, Bacar:LFCN-80, symbol LFCN-80
- added P6: CONN_01X02, Pin_Headers:Pin_Header_Straight_1x02, symbol CONN_01X02
- added P7: SMA, Bacar:SMA_Edge, symbol SMA
- added R10: oc, Resistors_SMD:R_0805_HandSoldering, symbol R
- added R11, R12: 0, Resistors_SMD:R_0805_HandSoldering, symbol R
Connections:
- wire segments 74 -> 88
Other:
- moved on the sheet: C1, C2, C3, C4, C5, C6, D1, J3, L1, L2, L3, L4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
